Commit message: [FEATURE] 1. Submodules of cartographer added 2. wheelchair_navigation added 3. wheelchair_cartographer added
[DESCRIPTION]
NA
[TESTING]
NA

[TRELLO CARD LINK]
NA
[REVIEWED BY]
NA

File: src/wheelchair_description/urdf/wheelchair.xacro (robot description, xacro)
@@ -27,5 +27,5 @@
         <origin xyz="0.1 0 0" rpy=" 0 0 0"/>
         <geometry>
-          <box size="0.75 0.40 0.60"/>
+          <box size="0.75 0.60 0.60"/>
         </geometry>
     <material name="black"/>
@@ -46,8 +46,7 @@
                       iyy="0.1000000042" iyz="0"
                       izz="0.1000000040"
-                      radius="0.29" length="0.06"
+                      radius="0.155" length="0.06"
                       radius_2="0.0028" length_2 ="0.005"
                       material="grey"/>
-                      <!-- filename="package://wheelchair_description/meshes/rm100_isg_wheel.dae" scale="1 1 1"/> -->
     <!--joint between chassis and Left wheel-->
         <w_joint name="chassis_to_left_wheel"
@@ -56,5 +55,5 @@
                  limit_e="100" limit_v="20"
                  damping="1.0" friction="200000.0"
-                 origin_rpy="-1.57 0 0" origin_xyz="-0.22 0.32 -0.15"
+                 origin_rpy="-1.57 0 0" origin_xyz="-0.22 0.28 -0.285"
                  parent="chassis" child="left_wheel"/>
       <!-- inertia values are added by 0.1 in both left and right wheel to avoid collapsing of model in gazebo-->
@@ -67,8 +66,7 @@
                        iyy="0.1000000042" iyz="0"
                        izz="0.1000000040"
-                       radius="0.29" length="0.06"
+                       radius="0.155" length="0.06"
                        radius_2="0.0028" length_2 ="0.005"
                        material="grey"/>
-                      <!-- filename="package://wheelchair_description/meshes/rm100_isg_wheel.dae" scale="1 1 1"/> -->
     <w_joint name="chassis_to_right_wheel"
              type="continuous"
@@ -77,5 +75,5 @@
              limit_e="100" limit_v="20"
              damping="1.0" friction="200000.0"
-             origin_rpy="-1.57 0 0" origin_xyz="-0.22 -0.27 -0.15"
+             origin_rpy="-1.57 0 0" origin_xyz="-0.22 -0.32 -0.285"
              parent="chassis" child="right_wheel" />
     <!--Caster 1,2 and there joints with Base Link-->
@@ -160,5 +158,5 @@
              origin_rpy="0 0 0" origin_xyz="0.23 0 -0.15"
              parent="chassis" child="lidar_base_rod" />
-<!--RP Lidar-->
+<!--Lidar-->
   <m_link_cylinder name="rplidar"
                    origin_rpy="0 0 0" origin_xyz="0 0 0"
@@ -169,5 +167,5 @@
                    material="black"
                    filename="package://wheelchair_description/meshes/rplidar.dae" scale="1 1 1"/>
-<!-- joint between chassis and rplidar -->
+<!-- joint between chassis and lidar -->
       <f_joint name="chassis_to_rplidar"
                type="fixed"
@@ -177,5 +175,5 @@
 <!--Real_Sense-->
       <sensor_d435 parent="base_link">
-        <origin xyz="-0.23 0 0.660" rpy="0 0 0"/>
+        <origin xyz="-0.23 0 0.860" rpy="0 0 0"/>
       </sensor_d435>
     <!--Gazebo Plugin-->

File: src/wheelchair_description/urdf/wheelchair_gazebo.xacro (robot description, xacro)
@@ -5,6 +5,6 @@
     <plugin name="differential_drive_controller" filename="libgazebo_ros_diff_drive.so">
       <alwaysOn>true</alwaysOn>
-      <commandTopic>wheelchair/cmd_vel</commandTopic>
-      <odometryTopic>wheelchair/odom</odometryTopic>
+      <commandTopic>diff/cmd_vel</commandTopic>
+      <odometryTopic>odom</odometryTopic>
       <odometryFrame>odom</odometryFrame>
       <odometrySource>world</odometrySource>
@@ -18,6 +18,6 @@
       <leftJoint>chassis_to_left_wheel</leftJoint>
       <rightJoint>chassis_to_right_wheel</rightJoint>
-      <wheelSeparation>0.420</wheelSeparation>
-      <wheelDiameter>0.1332</wheelDiameter>
+      <wheelSeparation>0.480</wheelSeparation>
+      <wheelDiameter>0.31</wheelDiameter>
       <wheelAcceleration>1</wheelAcceleration>
       <wheelTorque>40</wheelTorque>
@@ -27,21 +27,23 @@
   <!--Gazebo related physics values of left wheel joint-->
   <gazebo reference="chassis_to_left_wheel">
-    <mu1>0.1</mu1>
-    <mu2>0.1</mu2>
-    <kp>500000.0</kp>
-    <kd>10.0</kd>
-    <minDepth>0.001</minDepth>
-    <maxVel>0.1</maxVel>
-    <fdir1>1 0 0</fdir1>
+      <mu1 value="10000.0" />
+      <mu2 value="10000.0" />
+      <fdir1 value="0 0 1" />
+      <kp value="300" />  <!--500000-->
+      <kd value="10" />  <!--10-->
+      <ki value="200"/>
+      <maxVel value="2.0" />
+      <minDepth value="0.0001" />
   </gazebo>
   <!--Gazebo related physics values of right wheel joint-->
   <gazebo reference="chassis_to_right_wheel">
-    <mu1>0.1</mu1>
-    <mu2>0.1</mu2>
-    <kp>500000.0</kp>
-    <kd>10.0</kd>
-    <minDepth>0.001</minDepth>
-    <maxVel>0.1</maxVel>
-    <fdir1>1 0 0</fdir1>
+      <mu1 value="10000.0" />
+      <mu2 value="10000.0" />
+      <fdir1 value="0 0 1" />
+      <kp value="300" />
+      <kd value="10" />
+      <ki value="200" />
+      <maxVel value="2.0" />
+      <minDepth value="0.0001" />
   </gazebo>
   <gazebo reference="chassis">
@@ -49,20 +51,21 @@
   </gazebo>
   <gazebo reference="caster1">
-    <mu1>0.1</mu1>
-    <mu2>0.1</mu2>
+    <material>Gazebo/White</material>
+    <mu1>0.0</mu1>
+    <mu2>0.0</mu2>
+    <fdir1>0 0 0</fdir1>
     <kp>1000000.0</kp>
     <kd>100.0</kd>
     <minDepth>0.001</minDepth>
     <maxVel>1.0</maxVel>
-    <material>Gazebo/FlatBlack</material>
   </gazebo>
   <gazebo reference="caster2">
-    <mu1>0.1</mu1>
-    <mu2>0.1</mu2>
+    <material>Gazebo/White</material>
+    <mu1>0.0</mu1>
+    <mu2>0.0</mu2>
     <kp>1000000.0</kp>
     <kd>100.0</kd>
     <minDepth>0.001</minDepth>
     <maxVel>1.0</maxVel>
-    <material>Gazebo/FlatBlack</material>
   </gazebo>
     <gazebo reference="rod1">
@@ -95,5 +98,5 @@
         <range>
           <min>0.2</min>
-          <max>6.0</max>
+          <max>8.0</max>
           <resolution>0.01</resolution>
         </range>
@@ -109,86 +112,8 @@
       </ray>
       <plugin name="gazebo_ros_head_rplidar_controller" filename="libgazebo_ros_gpu_laser.so">
-        <topicName>wheelchair/scan</topicName>
+        <topicName>scan</topicName>
         <frameName>rplidar</frameName>
       </plugin>
     </sensor>
   </gazebo>
-  <gazebo reference="hokuyo_front">
-   <sensor type="ray" name="head_hokuyo_sensor1">
-    <pose>0 0 0 0 0 0</pose>
-    <always_on>1</always_on>
-    <update_rate>20</update_rate>
-    <visualize>false</visualize>
-    <ray>
-      <scan>
-        <horizontal>
-          <!-- The URG-04LX-UG01  has  683 steps with 0.35139 Degree resolution -->
-          <resolution>1</resolution>
-          <max_angle>1.658</max_angle> <!-- 120 Degree -->
-          <min_angle>-1.658</min_angle> <!-- -120 Degree -->
-          <!--max_angle>3.14</max_angle--> <!-- 120 Degree -->
-          <!--min_angle>-3.14</min_angle--> <!-- -120 Degree -->
-          <samples>720</samples>
-        </horizontal>
-      </scan>
-      <range>
-        <min>0.15</min>
-        <max>30.0</max>
-        <resolution>0.01</resolution>
-      </range>
-      <noise>
-        <type>gaussian</type>
-        <!-- Noise parameters based on published spec for Hokuyo laser
-             achieving "+-30mm" accuracy at range < 10m.  A mean of 0.0m and
-             stddev of 0.01m will put 99.7% of samples within 0.03m of the true
-             reading. -->
-        <mean>0.0</mean>
-        <stddev>0.01</stddev>
-      </noise>
-    </ray>
-    <plugin name="gazebo_ros_head_hokuyo_controller" filename="libgazebo_ros_laser.so">
-      <topicName>/wheelchair/scan_filtered1</topicName>
-      <frameName>hokuyo_front</frameName>
-    </plugin>
-   </sensor>
-  </gazebo>
-  <gazebo reference="hokuyo_back">
-   <sensor type="ray" name="head_hokuyo_sensor2">
-    <pose>0 0 0 0 0 0</pose>
-    <update_rate>20</update_rate>
-    <always_on>1</always_on>
-    <visualize>false</visualize>
-    <ray>
-      <scan>
-        <horizontal>
-          <!-- The URG-04LX-UG01  has  683 steps with 0.35139 Degree resolution -->
-          <resolution>1</resolution>
-          <max_angle>1.658</max_angle> <!-- 120 Degree -->
-          <min_angle>-1.658</min_angle> <!-- -120 Degree -->
-          <!--max_angle>3.14</max_angle--> <!-- 120 Degree -->
-          <!--min_angle>-3.14</min_angle--> <!-- -120 Degree -->
-          <samples>720</samples>
-        </horizontal>
-      </scan>
-      <range>
-        <min>0.15</min>
-        <max>30</max>
-        <resolution>0.01</resolution>
-      </range>
-      <noise>
-        <type>gaussian</type>
-        <!-- Noise parameters based on published spec for Hokuyo laser
-             achieving "+-30mm" accuracy at range < 10m.  A mean of 0.0m and
-             stddev of 0.01m will put 99.7% of samples within 0.03m of the true
-             reading. -->
-        <mean>0.0</mean>
-        <stddev>0.01</stddev>
-      </noise>
-    </ray>
-    <plugin name="gazebo_ros_head_hokuyo_controller" filename="libgazebo_ros_laser.so">
-      <topicName>/wheelchair/scan_filtered2</topicName>
-      <frameName>hokuyo_back</frameName>
-    </plugin>
-   </sensor>
-  </gazebo>
 </robot>
